File: usb-console.kicad_sch (KiCad schematic)
At the start: 0 parts

Commit message: [#1] WIP: Change components to ones from the global library, refactor schematic
Parts:
- added C2, C5: C-100n-0402, DW-footprints:C_0402_1005Metric, symbol DW-capacitors:C-100n-0402
- added D3: PUSB3F96X, DW-footprints:DFN2510A-10, symbol DW-TVS:PUSB3F96X
- added J4: USB-C-receptacle-16P_USB-310F-B-SU, DW-footprints:USB-C-receptacle-16P_USB-310F-B-SU, symbol DW-connectors:USB-C-receptacle-16P_USB-310F-B-SU
- added R21, R6: R-5k1-0402, DW-footprints:R_0402_1005Metric, symbol DW-resistors:R-5k1-0402
- added R5: R-330r-0402, DW-footprints:R_0402_1005Metric, symbol DW-resistors:R-330r-0402
Connections:
- new net: C2.2, J4.S1 (SHIELD), R5.2
- new net CC1: D3.5 (CH4), D3.6 (CH4), J4.A5 (CC1), R6.2
- new net CC2: D3.4 (CH3), D3.7 (CH3), J4.B5 (CC2), R21.2
- new net DEBUG_CONSOLE_VOUT: C5.2, J4.A4 (VBUS), J4.A9 (VBUS), J4.B4 (VBUS), J4.B9 (VBUS)
- new net GND: C2.1, C5.1, D3.3 (GND), D3.8 (GND), J4.A1 (GND), J4.A12 (GND), J4.B1 (GND), J4.B12 (GND), R21.1, R5.1, R6.1
- new net USB_PORT.D+: D3.2 (CH2), D3.9 (CH2), J4.A6 (D+), J4.B6 (D+)
- new net USB_PORT.D-: D3.1 (CH1), D3.10 (CH1), J4.A7 (D-), J4.B7 (D-)
- no-connect marks 0 -> 2
