File: usb-console.kicad_sch (KiCad schematic)
At the start: 31 parts, among them J11 USB-C_USB-310F-B-SU, U5 FT230XQ-R, U6 NTS0102DP

Commit message: [#3] Re-annotate schematic
Parts:
- renumbered C25 to C48, C26 to C49, C27 to C50, C28 to C51, C29 to C52, C30 to C53, C31 to C54, C32 to C55, D16 to D12, D17 to D13, D18 to D14, D19 to D15, D20 to D16, J11 to J10, R33 to R43, R34 to R44, R35 to R45, R36 to R46, R37 to R47, R38 to R48, R39 to R49, R40 to R50, R41 to R51, R42 to R52, TP9 to TP10, TP10 to TP11, TP11 to TP12, TP12 to TP13, TP13 to TP14, U6 to U10, U5 to U9
