File: usb.kicad_sch (KiCad schematic)
At the start: 22 parts, among them J8 USB-A_USB-303WSD-BRY, J9 USB-C_TYPE-C_16PLT-H6.5, U3 AP22615AWU-7

Commit message: [#3] Re-annotate schematic
Parts:
- renumbered C14 to C41, C15 to C42, C16 to C43, C17 to C44, C18 to C45, C19 to C46, C20 to C47, D9 to D10, D27 to D6, D8 to D7, D12 to D8, D10 to D9, R26 to R38, R27 to R39, R28 to R40, R29 to R41, R30 to R42, TP8 to TP9, U3 to U8
