File: pcb/cm5.kicad_sch (KiCad schematic)
At the start: 35 parts, among them J2 JST_SH_1x3_BM03B-SRSS-TB-LF-SN, J3 CM5_1-100_3mm-stack, J4 CM5_101-200_3mm-stack, J5 JST_SH_1x4_BM04B-SRSS-TB-LF-SN, SW1 SW_TL2243

Commit message: [#5] Refactor the schematic
Other:
- note added: "FAN CONNECTOR"
- note added: "MECHANICAL"
- note added: "RASPBERRY PI COMPUTE MODULE 5"
- moved on the sheet: A1, BT1, D2, D3, H1, H2, H3, H4, J2, J3, J4, J5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
